File: eagle/project/ETC_module.brd (EAGLE design)
At the start: 101.3 x 81.3 mm, 104 parts, among them IC1 LM358, P12-23 P12-23, Q2 MOSFET-PCHANNELFQP27P06, U1 V_REG_317SMD

Commit message: update to fix reverse polarity protection
FLIP DS  on FET, only done on ETC schematic
Connections:
- removed net N$13: BAT_CONN.1, Q2.2, U$1.K
- new net N$58: BAT_CONN.1, Q2.3, U$1.K
- net +12V: now also Q2.2; no longer Q2.3
Routing:
- net N$13: track 24.1 -> 0.00 mm
- net N$7: track 12.4 -> 7.79 mm
- net +12V: track 191.2 -> 187.6 mm
Changed lines of the file:
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@@
 </signal>
 <signal name="+12V">
-<contactref element="Q2" pad="3"/>
 <contactref element="10VZENER" pad="C"/>
 <contactref element="ISOPOW" pad="2"/>
@@
 <wire x1="90.17" y1="50.8" x2="91.44" y2="49.53" width="1.27" layer="1"/>
 <wire x1="91.44" y1="49.53" x2="93.345" y2="49.53" width="1.27" layer="1"/>
-<wire x1="93.345" y1="49.53" x2="95.885" y2="52.07" width="1.27" layer="1"/>
 <wire x1="90.17" y1="51.29" x2="88.41" y2="51.29" width="1.27" layer="1"/>
 <wire x1="88.41" y1="51.29" x2="86.36" y2="53.34" width="1.27" layer="1"/>
@@
 <wire x1="38.1" y1="65.532" x2="42.164" y2="61.468" width="1.016" layer="1"/>
 <wire x1="42.164" y1="61.468" x2="47.752" y2="61.468" width="1.016" layer="1"/>
+<contactref element="Q2" pad="2"/>
+<wire x1="93.345" y1="49.53" x2="95.885" y2="54.61" width="0" layer="19" extent="1-1"/>
 </signal>
 <signal name="N$6">
@@
 <wire x1="67.31" y1="68.58" x2="68.428" y2="68.58" width="0.635" layer="1"/>
 <wire x1="68.428" y1="68.58" x2="68.58" y2="68.732" width="0.635" layer="1"/>
-</signal>
-<signal name="N$13">
-<contactref element="BAT_CONN" pad="1"/>
-<contactref element="Q2" pad="2"/>
-<wire x1="95.25" y1="40.64" x2="99.06" y2="44.45" width="1.27" layer="1"/>
-<wire x1="99.06" y1="44.45" x2="99.06" y2="53.34" width="1.27" layer="1"/>
-<wire x1="99.06" y1="53.34" x2="97.79" y2="54.61" width="1.27" layer="1"/>
-<wire x1="97.79" y1="54.61" x2="95.885" y2="54.61" width="1.27" layer="1"/>
-<contactref element="U$1" pad="K"/>
-<wire x1="95.25" y1="40.64" x2="95.25" y2="36.3474" width="1.27" layer="16"/>
-<wire x1="95.25" y1="36.3474" x2="96.52" y2="35.0774" width="1.27" layer="16"/>
 </signal>
 <signal name="N$19">
@@
 <signal name="N$7">
 <contactref element="10VZENER" pad="A"/>
-<contactref element="Q2" pad="1"/>
 <contactref element="R5" pad="1"/>
-<wire x1="95.885" y1="57.15" x2="91.93" y2="57.15" width="1.27" layer="1"/>
 <wire x1="91.93" y1="57.15" x2="90.17" y2="55.39" width="1.27" layer="1"/>
 <wire x1="98.577" y1="61.595" x2="98.577" y2="59.207" width="1.27" layer="1"/>
 <wire x1="98.577" y1="59.207" x2="96.52" y2="57.15" width="1.27" layer="1"/>
-<wire x1="96.52" y1="57.15" x2="95.885" y2="57.15" width="1.27" layer="1"/>
+<contactref element="Q2" pad="1"/>
+<wire x1="95.885" y1="57.15" x2="96.52" y2="57.15" width="0" layer="19" extent="1-1"/>
+<wire x1="91.93" y1="57.15" x2="95.885" y2="57.15" width="0" layer="19" extent="1-1"/>
 </signal>
 <signal name="N$16">
@@
 <wire x1="56.896" y1="47.498" x2="57.912" y2="47.498" width="1.016" layer="1"/>
 </signal>
+<signal name="N$58">
+<contactref element="Q2" pad="3"/>
+<contactref element="BAT_CONN" pad="1"/>
+<contactref element="U$1" pad="K"/>
+<wire x1="95.25" y1="40.64" x2="95.885" y2="52.07" width="0" layer="19" extent="1-1"/>
+<wire x1="96.52" y1="35.0774" x2="95.25" y2="40.64" width="0" layer="19" extent="16-16"/>
+</signal>
 </signals>

Commit message: update before comp
Updates
Connections:
- net +12V: now also Q2.3; no longer Q2.2
- net N$58: now also Q2.2; no longer Q2.3
Changed lines of the file:
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@@
 <wire x1="38.1" y1="65.532" x2="42.164" y2="61.468" width="1.016" layer="1"/>
 <wire x1="42.164" y1="61.468" x2="47.752" y2="61.468" width="1.016" layer="1"/>
-<contactref element="Q2" pad="2"/>
-<wire x1="93.345" y1="49.53" x2="95.885" y2="54.61" width="0" layer="19" extent="1-1"/>
+<contactref element="Q2" pad="3"/>
+<wire x1="93.345" y1="49.53" x2="95.885" y2="52.07" width="0" layer="19" extent="1-1"/>
 </signal>
 <signal name="N$6">
@@
 </signal>
 <signal name="N$58">
-<contactref element="Q2" pad="3"/>
 <contactref element="BAT_CONN" pad="1"/>
 <contactref element="U$1" pad="K"/>
-<wire x1="95.25" y1="40.64" x2="95.885" y2="52.07" width="0" layer="19" extent="1-1"/>
+<contactref element="Q2" pad="2"/>
+<wire x1="95.25" y1="40.64" x2="95.885" y2="54.61" width="0" layer="19" extent="1-1"/>
 <wire x1="96.52" y1="35.0774" x2="95.25" y2="40.64" width="0" layer="19" extent="16-16"/>
 </signal>
